Commit message: trainning for stepping up the stairs

File: resources/robots/T1Bot/train_asset/t1_s_May11_09-55-12_v1.urdf (robot description, URDF)
Before this commit: robot fdrobot_t1, 15 links, 14 joints
Joints:
- joint leg_left_hipp: limit lower=-0.3 upper=1.0 effort=200 velocity=5 -> lower=-0.3 upper=1.2 effort=200 velocity=5
- joint leg_left_knee: limit lower=-0.0 upper=1.0 effort=250 velocity=5 -> lower=-0.0 upper=1.5 effort=250 velocity=5
- joint leg_right_hipp: limit lower=-0.3 upper=1.0 effort=200 velocity=5 -> lower=-0.3 upper=1.2 effort=200 velocity=5
- joint leg_right_knee: limit lower=-0.0 upper=1.0 effort=250 velocity=5 -> lower=-0.0 upper=1.5 effort=250 velocity=5

File: resources/robots/T1Bot/urdf/t1_s.urdf (robot description, URDF)
Before this commit: robot fdrobot_t1, 15 links, 14 joints
Joints:
- joint leg_left_hipp: limit lower=-0.3 upper=1.0 effort=200 velocity=5 -> lower=-0.3 upper=1.2 effort=200 velocity=5
- joint leg_right_hipp: limit lower=-0.3 upper=1.0 effort=200 velocity=5 -> lower=-0.3 upper=1.2 effort=200 velocity=5
